File: minato/minato.kicad_pcb (KiCad board)
At the start: 2 copper layers, 211 parts, among them U1 Elite-C

Commit message: :sparkles: Layout basic keyboard switches
Parts:
- D1, D10, D100, D101, D102, D103, D104, D105, D11, D12, D13, D14, D15, D16, D17, D18, D19, D2, D20, D21, D22, D23, D24, D25, D26, D27, D28, D29, D3, D30, D31, D32, D33, D34, D35, D36, D37, D38, D39, D4, D40, D41, D42, D43, D44, D45, D46, D47, D48, D49, D5, D50, D51, D52, D53, D54, D55, D56, D57, D58, D59, D6, D60, D61, D62, D63, D64, D65, D66, D67, D68, D69, D7, D70, D71, D72, D73, D74, D75, D76, D77, D78, D79, D8, D80, D81, D82, D83, D84, D85, D86, D87, D88, D89, D9, D90, D91, D92, D93, D94, D95, D96, D97, D98, D99: moved to B.Cu
- MX2:10: value Ctrl -> Ctrl 1.25u
- MX2:11: value Win -> Win 1.25u
- MX3:10: value Alt -> Alt 1.25u
- MX9:5: value | -> | 1.5u
- U1: footprint Keebio-Parts.pretty:Elite-C -> Keebio-Parts.pretty:Elite-C-castellated-29pin
- moved D105 351.8 mm to (157.6, 350.9)
- moved D84 351.8 mm to (169.1, 350.9)
- moved D90 351.8 mm to (163.4, 350.9)
- moved MX9:6 347.4 mm to (397.7, 146.8)
- moved D81 345.7 mm to (169.1, 347.6)
- moved D87 345.7 mm to (163.4, 347.6)
- moved D91 345.7 mm to (157.6, 347.6)
- moved MX9:9 343.3 mm to (397.7, 165.9)
- moved MX9:10 342.9 mm to (378.6, 184.9)
- moved MX9:1 342.2 mm to (397.7, 89.7)
- moved MX9:11 341.3 mm to (397.7, 184.9)
- moved D78 339.6 mm to (169.1, 344.2)
- moved D85 339.6 mm to (163.4, 344.2)
- moved D89 339.6 mm to (157.6, 344.2)
- moved D74 333.5 mm to (169.1, 340.9)
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
Commit message: :sparkles: Add stabilizers
Parts:
- added REF**: MX-Alps_Switch_Cutout, Keebio-Parts.pretty:MX_Stabilizer_Cutout, B.Cu at (269.1, 185.7)
- added REF**: MX-Alps_Switch_Cutout, Keebio-Parts.pretty:MX_Stabilizer_Cutout, F.Cu at (173.8, 185.7)
- added REF**: MX_Stabilizer_Cutout-2u, Keebio-Parts.pretty:MX_Stabilizer_Cutout-2u, F.Cu at (369.1, 109.5)
- added REF**: MX_Stabilizer_Cutout-2u, Keebio-Parts.pretty:MX_Stabilizer_Cutout-2u, F.Cu at (366.7, 147.6)
- added REF**: MX_Stabilizer_Cutout-2u, Keebio-Parts.pretty:MX_Stabilizer_Cutout-2u, F.Cu at (123.8, 166.7)
- added REF**: MX_Stabilizer_Cutout-2u, Keebio-Parts.pretty:MX_Stabilizer_Cutout-2u, F.Cu at (45.2, 185.7)

Commit message: :sparkles: Revamp stabilizers
Parts:
- removed the REF** at (269.1, 185.7)
- removed the REF** at (173.8, 185.7)
- removed the REF** at (369.1, 109.5)
- removed the REF** at (366.7, 147.6)
- removed the REF** at (123.8, 166.7)
- removed the REF** at (45.2, 185.7)
- removed U1: Elite-C, Keebio-Parts.pretty:Elite-C-castellated-29pin
- added REF**: MX-Alps_Switch_Cutout, Keebio-Parts.pretty:MX_Stabilizer_Cutout, B.Cu at (278.6, 184.9)
- added REF**: MX-Alps_Switch_Cutout, Keebio-Parts.pretty:MX_Stabilizer_Cutout, F.Cu at (183.4, 184.9)
- added REF**: MX_Stabilizer_Cutout-2u, Keebio-Parts.pretty:MX_Stabilizer_Cutout-2u, F.Cu at (369.1, 108.7)
- added REF**: MX_Stabilizer_Cutout-2u, Keebio-Parts.pretty:MX_Stabilizer_Cutout-2u, F.Cu at (366.7, 146.8)
- added REF**: MX_Stabilizer_Cutout-2u, Keebio-Parts.pretty:MX_Stabilizer_Cutout-2u, F.Cu at (123.8, 165.9)
- added REF**: MX_Stabilizer_Cutout-2u, Keebio-Parts.pretty:MX_Stabilizer_Cutout-2u, F.Cu at (45.2, 184.9)
- moved MX3:11 9.53 mm to (240.5, 184.9)
- moved MX1:5 9.52 mm to (92.9, 127.8)
- moved MX1:9 9.52 mm to (92.9, 165.9)

Commit message: :sparkles: Rev. 1 Routing
Parts:
- removed the REF** at (278.6, 184.9)
- removed the REF** at (183.4, 184.9)
- removed the REF** at (369.1, 108.7)
- removed the REF** at (366.7, 146.8)
- removed the REF** at (123.8, 165.9)
- removed the REF** at (45.2, 184.9)
- added HOLE_M2.6: VAL**, keyboard_parts.pretty:HOLE_M2.6, F.Cu at (17.5, 18.3)
- added HOLE_M2.6: VAL**, keyboard_parts.pretty:HOLE_M2.6, F.Cu at (450.9, 18.3)
- added HOLE_M2.6: VAL**, keyboard_parts.pretty:HOLE_M2.6, F.Cu at (450.9, 129.4)
- added HOLE_M2.6: VAL**, keyboard_parts.pretty:HOLE_M2.6, F.Cu at (17.5, 129.4)
- added REF**: MX_Stabilizer_Cutout-2u, Keebio-Parts.pretty:MX_Stabilizer_Cutout-2u, F.Cu at (386.6, 45.2)
- added REF**: MX_Stabilizer_Cutout-2u, Keebio-Parts.pretty:MX_Stabilizer_Cutout-2u, F.Cu at (62.7, 121.4)
- added REF**: MX-Alps_Switch_Cutout, Keebio-Parts.pretty:MX_Stabilizer_Cutout, B.Cu at (296.1, 121.4)
- added REF**: MX-Alps_Switch_Cutout, Keebio-Parts.pretty:MX_Stabilizer_Cutout, F.Cu at (200.8, 121.4)
- added REF**: MX_Stabilizer_Cutout-2u, Keebio-Parts.pretty:MX_Stabilizer_Cutout-2u, F.Cu at (384.2, 83.3)
- added REF**: MX_Stabilizer_Cutout-2u, Keebio-Parts.pretty:MX_Stabilizer_Cutout-2u, F.Cu at (141.3, 102.4)
- added U1: Elite-C, Keebio-Parts.pretty:Elite-C-castellated-29pin-holes, F.Cu at (437.4, 34.1)
- moved D96 459.7 mm to (386.6, 31.8), turned to 90 degrees
- moved D100 459.7 mm to (406.4, 28.6), turned to 90 degrees
- moved D101 439.0 mm to (404.8, 50.7), turned to 90 degrees
- moved D97 428.3 mm to (381.8, 66.7), turned to 90 degrees
- moved D102 422.5 mm to (405.6, 69.8), turned to 90 degrees
- moved D80 420.3 mm to (329.4, 47.6), turned to 90 degrees
- moved D94 416.3 mm to (365.1, 85.7), turned to 90 degrees
- moved D103 405.6 mm to (405.6, 88.9), turned to 90 degrees
- moved D98 401.3 mm to (386.6, 108.0), turned to 90 degrees
- moved D92 400.0 mm to (368.3, 47.6), turned to 90 degrees
- moved D104 391.1 mm to (405.6, 104.8), turned to 90 degrees
- moved D95 390.4 mm to (367.5, 123.8), turned to 90 degrees
- moved D99 385.4 mm to (386.6, 126.9), turned to 90 degrees
- moved D91 381.9 mm to (367.5, 28.6), turned to 90 degrees
- moved D85 363.2 mm to (348.5, 31.8), turned to 90 degrees
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Routing:
- net Col3: track 0.00 -> 608.4 mm, vias 0 -> 12
- net Col0: track 0.00 -> 584.9 mm, vias 0 -> 7
- net Col1: track 0.00 -> 531.6 mm, vias 0 -> 7
- net Col2: track 0.00 -> 524.4 mm, vias 0 -> 7
- net Row9: track 0.00 -> 511.9 mm, vias 0 -> 17
- net Row10: track 0.00 -> 507.5 mm
- net Row11: track 0.00 -> 498.8 mm, vias 0 -> 12
- net Row8: track 0.00 -> 488.4 mm
- net Row7: track 0.00 -> 479.8 mm, vias 0 -> 16
- net Row6: track 0.00 -> 463.6 mm
- net Row5: track 0.00 -> 462.2 mm, vias 0 -> 18
- net Row1: track 0.00 -> 451.9 mm, vias 0 -> 20
- net Row4: track 0.00 -> 441.8 mm
- net Row3: track 0.00 -> 438.4 mm, vias 0 -> 18
- net Row0: track 0.00 -> 428.5 mm
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Other:
- board outline added: 438.1 x 115.9 mm
- net class Matrix added: clearance 0.1778, trace_width 0.1778, via_dia 0.8, via_drill 0.4
- rule trace_min: 0.2 -> 0.1778
- board text added: "minato"
- board text added: "rev. 1 - 2/7/2020"

Commit message: :sparkles: Rev. 2 Routing
Parts:
- removed D1: 1N4148, Diode_SMD:D_SOD-123
- removed MX0:0: Macro1, keyswitches.pretty:Kailh_socket_MX
- removed the REF** at (386.6, 45.2)
- removed the REF** at (62.7, 121.4)
- removed the REF** at (296.1, 121.4)
- removed the REF** at (200.8, 121.4)
- removed the REF** at (384.2, 83.3)
- removed the REF** at (141.3, 102.4)
- added REF**: 6U, MX_Alps_Hybrid:MXOnly-6U, F.Cu at (248.4, 121.4)
- added REF**: Stabilizer_MX_2u, keyswitches.pretty:Stabilizer_MX_2u, F.Cu at (386.6, 45.2)
- added REF**: Stabilizer_MX_2u, keyswitches.pretty:Stabilizer_MX_2u, F.Cu at (384.2, 83.3)
- added REF**: Stabilizer_MX_2u, keyswitches.pretty:Stabilizer_MX_2u, F.Cu at (141.3, 102.4)
- added REF**: Stabilizer_MX_2u, keyswitches.pretty:Stabilizer_MX_2u, F.Cu at (62.7, 121.4)
- U1: footprint Keebio-Parts.pretty:Elite-C-castellated-29pin-holes -> Keebio-Parts.pretty:Elite-C-castellated-29pin; moved to B.Cu
- moved U1 386.8 mm to (50.8, 19.4)
- moved HOLE_M2.6 23.8 mm to (431.8, 3.97)
- moved HOLE_M2.6 23.8 mm to (36.5, 3.97)
- moved HOLE_M2.6 23.8 mm to (431.8, 143.7)
- moved HOLE_M2.6 23.8 mm to (36.5, 143.7)
- moved D94 19.3 mm to (384.2, 88.9), turned to 180 degrees
- moved D26 19.0 mm to (141.3, 108.0), turned to 180 degrees
- moved D92 18.5 mm to (386.6, 50.8), turned to 180 degrees
- moved D6 17.5 mm to (62.7, 127.0), turned to 180 degrees
- moved D21 10.4 mm to (110.7, 108.0), turned to 180 degrees
- moved D101 10.3 mm to (415.1, 50.7), turned to 180 degrees
- moved D27 10.3 mm to (131.8, 127.0), turned to 180 degrees
- moved D71 10.0 mm to (296.1, 88.9), turned to 180 degrees
- moved D68 10.0 mm to (300.8, 31.8), turned to 180 degrees
- moved D104 10.0 mm to (415.1, 108.0), turned to 180 degrees
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Routing:
- net Col0: track 584.9 -> 213.9 mm, vias 7 -> 0
- net Col1: track 531.6 -> 223.3 mm, vias 7 -> 2
- net Col2: track 524.4 -> 257.7 mm, vias 7 -> 2
- net Col9: track 314.6 -> 578.7 mm, vias 7 -> 2
- net Col6: track 208.1 -> 442.8 mm, vias 7 -> 2
- net Col7: track 290.3 -> 513.0 mm, vias 10 -> 4
- net Col5: track 186.7 -> 409.4 mm, vias 7 -> 2
- net Col3: track 608.4 -> 410.3 mm, vias 12 -> 2
- net Col8: track 381.6 -> 565.4 mm, vias 10 -> 4
- net Row0: track 428.5 -> 385.6 mm, vias 0 -> 11
- net Row1: track 451.9 -> 415.2 mm, vias 20 -> 12
- net Row3: track 438.4 -> 406.0 mm, vias 18 -> 9
- net Row7: track 479.8 -> 449.2 mm, vias 16 -> 8
- net Row5: track 462.2 -> 435.8 mm, vias 18 -> 9
- net Row11: track 498.8 -> 518.5 mm, vias 12 -> 6
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Other:
- board size 438.1 x 115.9 mm -> 400 x 144.5 mm

Commit message: :tada: Rev 1 initial design complete
Connections:
- U1 pad 23: Net-(U1-Pad23) -> GND
- U1 pad 3: Net-(U1-Pad3) -> GND
- U1 pad 4: Net-(U1-Pad4) -> GND
Routing:
- net GND: track 0.00 -> 35.3 mm
Other:
- board text added: "rev. 1 - 2/9/2020"
- board text removed: "rev. 1 - 2/7/2020"
Changed lines of the file:
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@@
     (thickness 1.6)
     (drawings 11)
-    (tracks 1220)
+    (tracks 1227)
     (zones 0)
     (modules 218)
-    (nets 134)
+    (nets 132)
   )
   (page A2)
@@
     (visible_elements 7FFFFFFF)
     (pcbplotparams
-      (layerselection 0x010fc_ffffffff)
+      (layerselection 0x010f0_ffffffff)
       (usegerberextensions false)
       (usegerberattributes false)
@@
       (outputformat 1)
       (mirror false)
-      (drillshape 1)
+      (drillshape 0)
       (scaleselection 1)
-      (outputdirectory ""))
+      (outputdirectory "../Gerbers"))
   )
   (net 0 "")
@@
   (net 126 Col9)
   (net 127 "Net-(U1-Pad24)")
-  (net 128 "Net-(U1-Pad23)")
-  (net 129 "Net-(U1-Pad22)")
-  (net 130 "Net-(U1-Pad21)")
-  (net 131 "Net-(U1-Pad4)")
-  (net 132 "Net-(U1-Pad3)")
-  (net 133 "Net-(U1-Pad2)")
+  (net 128 "Net-(U1-Pad22)")
+  (net 129 "Net-(U1-Pad21)")
+  (net 130 "Net-(U1-Pad2)")
+  (net 131 GND)
   (net_class Default "This is the default net class."
     (clearance 0.2)
@@
     (uvia_dia 0.3)
     (uvia_drill 0.1)
+    (add_net GND)
     (add_net "Net-(D10-Pad2)")
     (add_net "Net-(D100-Pad2)")
@@
     (add_net "Net-(U1-Pad21)")
     (add_net "Net-(U1-Pad22)")
-    (add_net "Net-(U1-Pad23)")
     (add_net "Net-(U1-Pad24)")
-    (add_net "Net-(U1-Pad3)")
-    (add_net "Net-(U1-Pad4)")
   )
   (net_class Matrix ""
@@
       (net 127 "Net-(U1-Pad24)"))
     (pad 23 smd rect (at -11.43 9.398 270) (size 2 3.25) (layers B.Cu B.Paste B.Mask)
-      (net 128 "Net-(U1-Pad23)"))
+      (net 131 GND))
     (pad 22 smd rect (at -8.89 9.398 270) (size 2 3.25) (layers B.Cu B.Paste B.Mask)
-      (net 129 "Net-(U1-Pad22)"))
+      (net 128 "Net-(U1-Pad22)"))
     (pad 21 smd rect (at -6.35 9.398 270) (size 2 3.25) (layers B.Cu B.Paste B.Mask)
-      (net 130 "Net-(U1-Pad21)"))
+      (net 129 "Net-(U1-Pad21)"))
     (pad 20 smd rect (at -3.81 9.398 270) (size 2 3.25) (layers B.Cu B.Paste B.Mask)
       (net 28 Row11))
@@
       (net 118 Col1))
     (pad 4 smd rect (at -6.35 -9.398 270) (size 2 3.25) (layers B.Cu B.Paste B.Mask)
-      (net 131 "Net-(U1-Pad4)"))
+      (net 131 GND))
     (pad 3 smd rect (at -8.89 -9.398 270) (size 2 3.25) (layers B.Cu B.Paste B.Mask)
-      (net 132 "Net-(U1-Pad3)"))
+      (net 131 GND))
     (pad 2 smd rect (at -11.43 -9.398 270) (size 2 3.25) (layers B.Cu B.Paste B.Mask)
-      (net 133 "Net-(U1-Pad2)"))
+      (net 130 "Net-(U1-Pad2)"))
     (pad 1 smd rect (at -13.97 -9.398 270) (size 2 3.25) (layers B.Cu B.Paste B.Mask)
       (net 117 Col0))
@@
     (arrow2b (pts (xy 56.753125 90.884375) (xy 56.371229 92.095596)))
   )
-  (gr_text "rev. 1 - 2/7/2020" (at 216.69375 122.316875) (layer F.SilkS)
+  (gr_text "rev. 1 - 2/9/2020" (at 216.69375 122.316875) (layer F.SilkS)
     (effects (font (size 1 1) (thickness 0.15)))
   )
@@
   (segment (start 395.2875 55.5625) (end 394.887501 55.962499) (width 0.1778) (layer F.Cu) (net 126))
   (segment (start 394.887501 55.962499) (end 46.040624 55.962499) (width 0.1778) (layer F.Cu) (net 126))
+  (segment (start 58.323 10.556875) (end 60.198 10.556875) (width 0.25) (layer B.Cu) (net 131))
+  (segment (start 43.277 8.016875) (end 45.817 10.556875) (width 0.25) (layer B.Cu) (net 131))
+  (segment (start 45.817 10.556875) (end 58.323 10.556875) (width 0.25) (layer B.Cu) (net 131))
+  (segment (start 41.402 8.016875) (end 43.277 8.016875) (width 0.25) (layer B.Cu) (net 131))
+  (segment (start 58.323 13.096875) (end 55.783 10.556875) (width 0.25) (layer B.Cu) (net 131))
+  (segment (start 55.783 10.556875) (end 45.817 10.556875) (width 0.25) (layer B.Cu) (net 131))
+  (segment (start 60.198 13.096875) (end 58.323 13.096875) (width 0.25) (layer B.Cu) (net 131))
 )

Commit message: :tada: Rev. 1 production
Parts:
- moved D100 23.0 mm to (398.5, 47.6)
- moved D101 23.0 mm to (398.5, 66.6)
- moved D102 23.0 mm to (398.5, 85.7)
- moved D103 23.0 mm to (398.5, 104.8)
- moved D104 23.0 mm to (398.5, 123.8)
- moved D105 23.0 mm to (398.5, 142.9)
- moved D71 23.0 mm to (279.4, 104.8)
- moved D73 23.0 mm to (303.2, 47.6)
- moved D74 23.0 mm to (303.2, 66.7)
- moved D83 23.0 mm to (327.0, 123.8)
- moved D90 23.0 mm to (338.9, 142.9)
- moved D93 23.0 mm to (350.8, 85.7)
- moved D97 23.0 mm to (374.6, 85.7)
- moved MX6:7 23.0 mm to (279.4, 99.2)
- moved MX7:0 23.0 mm to (303.2, 42.1)
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Other:
- board size 400 x 144.5 mm -> 400.1 x 144.5 mm

Commit message: :construction: Add STM32F103 schematic
Parts:
- removed HOLE_M2.6 (x4): VAL**, keyboard_parts.pretty:HOLE_M2.6
- removed U1: Elite-C, Keebio-Parts.pretty:Elite-C-castellated-29pin
- added D1: 1N4148, Diode_SMD:D_SOD-123, B.Cu at (29.0, 33.7)
- added HOLE_M3: VAL**, keyboard_parts.pretty:HOLE_M3, F.Cu at (414.7, 20.2)
- added HOLE_M3: VAL**, keyboard_parts.pretty:HOLE_M3, F.Cu at (414.7, 159.1)
- added HOLE_M3: VAL**, keyboard_parts.pretty:HOLE_M3, F.Cu at (20.2, 159.1)
- added HOLE_M3: VAL**, keyboard_parts.pretty:HOLE_M3, F.Cu at (20.2, 20.2)
- added MX0:0: Macro1, keyswitches.pretty:Kailh_socket_MX, F.Cu at (36.5, 42.1)
- added U2: STM32F103C8Tx, Package_QFP:LQFP-48_7x7mm_P0.5mm, F.Cu at (65.3, 19.5)
- moved D63 15.8 mm to (257.6, 33.7), turned to 270 degrees
- moved D64 15.8 mm to (257.6, 52.8), turned to 270 degrees
- moved D96 15.8 mm to (371.9, 33.7), turned to 270 degrees
- moved D2 15.8 mm to (29.0, 52.8), turned to 270 degrees
- moved D22 15.8 mm to (105.2, 33.7), turned to 270 degrees
- moved D23 15.8 mm to (105.2, 52.8), turned to 270 degrees
- moved D31 15.8 mm to (143.3, 33.7), turned to 270 degrees
- moved D32 15.8 mm to (143.3, 52.8), turned to 270 degrees
- moved D43 15.8 mm to (181.4, 33.7), turned to 270 degrees
- moved D44 15.8 mm to (181.4, 52.8), turned to 270 degrees
- moved D12 15.8 mm to (67.1, 33.7), turned to 270 degrees
- moved D13 15.8 mm to (67.1, 52.8), turned to 270 degrees
- moved D53 15.8 mm to (219.5, 33.7), turned to 270 degrees
- moved D54 15.8 mm to (219.5, 52.8), turned to 270 degrees
- moved D73 15.8 mm to (295.7, 33.7), turned to 270 degrees
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Routing:
- net Col8: track 565.4 -> 0.00 mm, vias 4 -> 0
- net Row11: track 518.5 -> 0.00 mm, vias 6 -> 0
- net Col7: track 513.0 -> 0.00 mm, vias 4 -> 0
- net Row9: track 508.3 -> 0.00 mm, vias 11 -> 0
- net Row10: track 489.5 -> 0.00 mm, vias 6 -> 0
- net Row8: track 480.9 -> 0.00 mm, vias 9 -> 0
- net Row6: track 476.0 -> 0.00 mm, vias 9 -> 0
- net Row4: track 454.0 -> 0.00 mm, vias 10 -> 0
- net Row7: track 449.2 -> 0.00 mm, vias 8 -> 0
- net Col6: track 442.8 -> 0.00 mm, vias 2 -> 0
- net Row5: track 435.8 -> 0.00 mm, vias 9 -> 0
- net Col3: track 410.3 -> 0.00 mm, vias 2 -> 0
- net Col5: track 409.4 -> 0.00 mm, vias 2 -> 0
- net Col9: track 578.7 -> 201.1 mm, vias 2 -> 10
- net Col4: track 372.6 -> 0.00 mm, vias 2 -> 0
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